File: Printed Circuit Board/gimbal.sch (KiCad schematic (older format))
At the start: 2 parts, among them J5 Conn_01x03_Male, J6 Conn_01x03_Male

Commit message: PCB: physical board prototype
Parts:
- J5, J6: footprint (none) -> Connector_PinHeader_2.54mm:PinHeader_1x03_P2.54mm_Vertical
Changed lines of the file:
@@
 F 0 "J6" H 6908 3681 50  0000 C CNN
 F 1 "Conn_01x03_Male" H 6908 3590 50  0000 C CNN
-F 2 "" H 6800 3400 50  0001 C CNN
+F 2 "Connector_PinHeader_2.54mm:PinHeader_1x03_P2.54mm_Vertical" H 6800 3400 50  0001 C CNN
 F 3 "~" H 6800 3400 50  0001 C CNN
 	1    6800 3400
@@
 F 0 "J5" H 5658 3681 50  0000 C CNN
 F 1 "Conn_01x03_Male" H 5658 3590 50  0000 C CNN
-F 2 "" H 5550 3400 50  0001 C CNN
+F 2 "Connector_PinHeader_2.54mm:PinHeader_1x03_P2.54mm_Vertical" H 5550 3400 50  0001 C CNN
 F 3 "~" H 5550 3400 50  0001 C CNN
 	1    5550 3400

Commit message: PCB physical board
Parts:
- J5: value Conn_01x03_Male -> horizontal servo connector
- J6: value Conn_01x03_Male -> vertical servo connector
Changed lines of the file:
@@
 AR Path="/6039BD63/6039FDDF" Ref="J6"  Part="1"
 F 0 "J6" H 6908 3681 50  0000 C CNN
-F 1 "Conn_01x03_Male" H 6908 3590 50  0000 C CNN
+F 1 "vertical servo connector" H 6908 3590 50  0000 C CNN
 F 2 "Connector_PinHeader_2.54mm:PinHeader_1x03_P2.54mm_Vertical" H 6800 3400 50  0001 C CNN
 F 3 "~" H 6800 3400 50  0001 C CNN
@@
 AR Path="/6039BD63/6039FDE5" Ref="J5"  Part="1"
 F 0 "J5" H 5658 3681 50  0000 C CNN
-F 1 "Conn_01x03_Male" H 5658 3590 50  0000 C CNN
+F 1 "horizontal servo connector" H 5658 3590 50  0000 C CNN
 F 2 "Connector_PinHeader_2.54mm:PinHeader_1x03_P2.54mm_Vertical" H 5550 3400 50  0001 C CNN
 F 3 "~" H 5550 3400 50  0001 C CNN
