File: Printed Circuit Board/turret_pcb.kicad_pcb (KiCad board)
At the start: 2 copper layers, 24 parts, among them J1 Conn_02x20_Odd_Even, J10 Conn_01x03_Female, J11 Conn_02x03_Odd_Even, J2 speaker_connector, J3 speaker, J4 Conn_01x02_Female, J5 Conn_01x03_Male, J6 Conn_01x03_Male, J7 Conn_01x04_Male, J8 Conn_01x04_Male, J9 Conn_02x03_Odd_Even, Q2 2N2219

Commit message: PCB physical board
Parts:
- A1: value Pololu_Breakout_DRV8825 -> stepper driver DRV8825 (1)
- A2: value Pololu_Breakout_DRV8825 -> stepper driver DRV8825 (2)
- J1: moved to B.Cu
- J10: value Conn_01x03_Female -> motion detector connector
- J11: value Conn_02x03_Odd_Even -> stepper driver M jumper (2)
- J2: value speaker_connector -> speaker connector
- J4: value Conn_01x02_Female -> laser connector
- J5: value Conn_01x03_Male -> horizontal servo connector
- J6: value Conn_01x03_Male -> vertical servo connector
- J7: value Conn_01x04_Male -> stepper motor connector (1)
- J8: value Conn_01x04_Male -> stepper motor connector (2)
- J9: value Conn_02x03_Odd_Even -> stepper driver M jumper (1); footprint Connector_PinSocket_2.54mm:PinSocket_2x03_P2.54mm_Horizontal -> Connector_PinSocket_2.54mm:PinSocket_2x03_P2.54mm_Vertical
- Q2: value 2N2219 -> laser transistor
- R7: value R -> SLP_R_2
- moved C2 123.1 mm to (104.1, 108.0), turned to 90 degrees
- moved J3 118.8 mm to (94.0, 92.7)
- moved R7 110.7 mm to (199.4, 94.0)
- moved RST_R_2 110.3 mm to (205.7, 96.5)
- moved R1 107.5 mm to (113.0, 101.9), turned to 270 degrees
- moved R2 106.6 mm to (108.0, 101.8), turned to 90 degrees
- moved J2 105.0 mm to (104.1, 90.2)
- moved C1 103.2 mm to (113.0, 97.8), turned to 180 degrees
- moved J10 103.1 mm to (141.0, 101.6), turned to 180 degrees
- moved SLP_R_1 83.6 mm to (166.4, 94.0)
- moved RST_R_1 76.3 mm to (172.7, 96.5)
- moved J5 74.4 mm to (137.2, 96.5)
- moved J6 73.6 mm to (133.3, 96.5)
- moved A2 73.1 mm to (181.6, 88.9)
- moved V1 71.4 mm to (153.7, 116.8)
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- renumbered R3 to RST_R_1, R5 to RST_R_2, R4 to SLP_R_1, R6 to laser_R1
Connections:
- A1 pad 15: /GPIO27 -> /GPIO17
- A1 pad 16: /GPIO17 -> /GPIO27
- A2 pad 15: /GPIO10 -> /GPIO22
- A2 pad 16: /GPIO22 -> /GPIO10
- J11 pad 2: Net-(A2-Pad10) -> Net-(A2-Pad12)
- J11 pad 6: Net-(A2-Pad12) -> Net-(A2-Pad10)
- J9 pad 2: Net-(A1-Pad10) -> Net-(A1-Pad12)
- J9 pad 6: Net-(A1-Pad12) -> Net-(A1-Pad10)
Routing:
- net /5V: track 0.00 -> 233.6 mm
- net /5V_GND: track 0.00 -> 159.8 mm
- net /GPIO18: track 0.00 -> 59.8 mm, vias 0 -> 1
- net /12V_GND: track 0.00 -> 50.8 mm
- net /12V: track 0.00 -> 44.4 mm
- net /GPIO22: track 0.00 -> 42.8 mm
- net /GPIO4: track 0.00 -> 40.1 mm, vias 0 -> 2
- net /GPIO10: track 0.00 -> 36.7 mm
- net /GPIO2: track 0.00 -> 24.7 mm
- net /GPIO3: track 0.00 -> 24.2 mm
- net /GPIO14: track 0.00 -> 23.7 mm
- net /GPIO17: track 0.00 -> 15.6 mm
- net Net-(C1-Pad1): track 0.00 -> 15.1 mm
- net Net-(A2-Pad13): track 0.00 -> 12.3 mm
- net /GPIO27: track 0.00 -> 12.0 mm
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
Commit message: KiCAD version updated 5 -> 6
Other:
- net class Default removed
